File: Hardware Files/ESP-ExtBoard/ESP-ExtBoard.kicad_pcb (KiCad board)
At the start: 2 copper layers, 72.6 x 58.4 mm, 8 parts, among them J1 PIN_HEADER, J2 PIN_HEADER_1x4, J3 PIN_HEADER, J4 PIN_HEADER, U1 ESP32-DEVKIT-V1, U2 BME280, U3 MPU6050, U4 SSD1306

Commit message: Starting V2.0
Parts:
- removed J1: PIN_HEADER, New_lib:PinHeader_1x06_P2.54mm_Vertical_1
- removed U1: ESP32-DEVKIT-V1, New_lib:MODULE_ESP32_DEVKIT_V1
- added J5: 502570-0893, New_lib:MOLEX_502570-0893, B.Cu at (100.8, 101.9)
- added J6: Micro-usb, New_lib:AMPHENOL_10118194-0001LF, F.Cu at (97.8, 114.8)
- added U5: ESP32-WROOM-32, RF_Module:ESP32-WROOM-32, F.Cu at (100.5, 80.7)
- added U6: CH340C, New_lib:SOIC127P600X180-16N, F.Cu at (97.2, 102.5)
- added U7: AMS1117-3.3, Package_TO_SOT_SMD:SOT-223-3_TabPin2, F.Cu at (107.8, 102.2)

Commit message: Added GPS Module
Parts:
- removed J2: PIN_HEADER_1x4, New_lib:PinHeader_1x04_P2.54mm_Vertical_1
- added J1: NEO-GPS, New_lib:NEO-GPS, F.Cu at (116.0, 78.5)
- U2, U3: moved to B.Cu
- moved J5 50.7 mm to (144.1, 75.2), turned to 90 degrees
- moved U2 22.8 mm to (148.5, 91.3), turned to 180 degrees
- moved U7 15.3 mm to (92.5, 101.0)
- moved U3 10.7 mm to (111.5, 91.2), turned to 180 degrees
- moved U6 6.49 mm to (103.5, 100.8)
- moved U5 6.20 mm to (100.4, 74.5)
- moved U4 3.76 mm to (127.4, 101.4)
Connections:
- U5 pad 1: Net-(U5-GND-Pad1) -> Earth
- U5 pad 10: unconnected-(U5-IO25-Pad10) -> /GPIO25
- U5 pad 11: unconnected-(U5-IO26-Pad11) -> /GPIO26
- U5 pad 12: unconnected-(U5-IO27-Pad12) -> /GPIO27
- U5 pad 13: unconnected-(U5-IO14-Pad13) -> /GPIO14
- U5 pad 15: Net-(U5-GND-Pad1) -> Earth
- U5 pad 2: unconnected-(U5-VDD-Pad2) -> +3.3V
- U5 pad 27: unconnected-(U5-IO16-Pad27) -> /UART2_RX
- U5 pad 28: unconnected-(U5-IO17-Pad28) -> /UART2_TX
- U5 pad 29: unconnected-(U5-IO5-Pad29) -> /VSPI_CS
- U5 pad 30: unconnected-(U5-IO18-Pad30) -> /VSPI_CLK
- U5 pad 31: unconnected-(U5-IO19-Pad31) -> /VSPI_MISO
- U5 pad 33: unconnected-(U5-IO21-Pad33) -> /I2C0_SDA
- U5 pad 34: unconnected-(U5-RXD0/IO3-Pad34) -> /UART0_RX
- U5 pad 35: unconnected-(U5-TXD0/IO1-Pad35) -> /UART0_TX
- U5 pad 36: unconnected-(U5-IO22-Pad36) -> /I2C0_SCL
- U5 pad 37: unconnected-(U5-IO23-Pad37) -> /VSPI_MOSI
- U5 pad 38: Net-(U5-GND-Pad1) -> Earth
- U5 pad 39: Net-(U5-GND-Pad1) -> Earth
- U5 pad 6: unconnected-(U5-IO34-Pad6) -> /GPIO34
- U5 pad 7: unconnected-(U5-IO35-Pad7) -> /GPIO35
- U5 pad 8: unconnected-(U5-IO32-Pad8) -> /GPIO32
- U5 pad 9: unconnected-(U5-IO33-Pad9) -> /GPIO33
- U6 pad 16: unconnected-(U6-VCC-Pad16) -> +3.3V
- U6 pad 2: unconnected-(U6-TXD-Pad2) -> /UART0_TX
- U6 pad 3: unconnected-(U6-RXD-Pad3) -> /UART0_RX
- U7 pad 1: unconnected-(U7-GND-Pad1) -> Earth
- U7 pad 2: unconnected-(U7-VO-Pad2) -> +3.3V
Routing:
- net +3.3V: track 154.7 -> 0.00 mm
- net /UART2_RX: track 77.0 -> 0.00 mm
- net /I2C0_SCL: track 75.1 -> 0.00 mm
- net /VSPI_MOSI: track 57.3 -> 0.00 mm
- net /I2C0_SDA: track 50.9 -> 0.00 mm
- net +5V: track 49.0 -> 0.00 mm
- net /VSPI_CS: track 40.8 -> 0.00 mm
- net /VSPI_CLK: track 40.8 -> 0.00 mm
- net /VSPI_MISO: track 39.7 -> 0.00 mm
- net /UART2_TX: track 36.6 -> 0.00 mm
- net /GPIO35: track 4.79 -> 0.00 mm
- net /GPIO33: track 4.79 -> 0.00 mm
- net /GPIO32: track 4.79 -> 0.00 mm
- net /GPIO34: track 4.79 -> 0.00 mm
- net /GPIO27: track 4.57 -> 0.00 mm
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Other:
- board text added: "ESP32 RX"
- board text added: "ESP32 TX"
- board text added: "GPS Module"
- board text added: "Z-ESP32 V2.0 Design by Guilherme Freire"
- board text removed: "GND VCC MISO MOSI CLK CS"
- board text removed: "SD CARD MODULE"
- board text removed: "UART2_RX"
- board text removed: "UART2_TX"
- board text removed: "Zephyr ESP32 Breakout Board v 1.0 Design by Guilherme Freire"
