File: Hardware Files/ESP-ExtBoard/ESP-ExtBoard.kicad_sch (KiCad schematic)
At the start: 8 parts, among them J1 PIN_HEADER, J2 PIN_HEADER_1x4, J3 PIN_HEADER, J4 PIN_HEADER, U1 ESP32-DEVKIT-V1, U2 BME280, U3 MPU6050, U4 SSD1306

Commit message: Starting V2.0
Parts:
- added J5: 502570-0893, New_lib:MOLEX_502570-0893, symbol New_Library:502570-0893
- added J6: Micro-usb, New_lib:AMPHENOL_10118194-0001LF, symbol New_Library:Micro-usb
- added U5: ESP32-WROOM-32, RF_Module:ESP32-WROOM-32, symbol RF_Module:ESP32-WROOM-32
- added U6: CH340C, New_lib:SOIC127P600X180-16N, symbol New_Library:CH340C
- added U7: AMS1117-3.3, Package_TO_SOT_SMD:SOT-223-3_TabPin2, symbol Regulator_Linear:AMS1117-3.3
Connections:
- new net: J6.S1 (SHIELD), J6.S2 (SHIELD), J6.S3 (SHIELD), J6.S4 (SHIELD), J6.S5 (SHIELD), J6.S6 (SHIELD)
- new net: U5.1 (GND), U5.15 (GND), U5.38 (GND), U5.39 (GND)
Changed lines of the file:
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@@
     (effects (font (size 1.27 1.27)) (justify right bottom))
+  )
+  (symbol (lib_id "New_Library:Micro-usb") (at 240.03 140.97 0) (unit 1)
+    (in_bom yes) (on_board yes) (dnp no) (fields_autoplaced)
+    (property "Reference" "J6" (at 246.38 139.7 0)
+      (effects (font (size 1.27 1.27)) (justify left))
+    )
+    (property "Value" "Micro-usb" (at 246.38 142.24 0)
+      (effects (font (size 1.27 1.27)) (justify left))
+    )
+    (property "Footprint" "New_lib:AMPHENOL_10118194-0001LF" (at 240.03 140.97 0)
+      (effects (font (size 1.27 1.27)) (justify bottom) hide)
+    )
+    (property "Datasheet" "" (at 240.03 140.97 0)
+      (effects (font (size 1.27 1.27)) hide)
+    )
+    (property "PARTREV" "D" (at 240.03 140.97 0)
+      (effects (font (size 1.27 1.27)) (justify bottom) hide)
+    )
+    (property "STANDARD" "Manufacturer Recommendations" (at 240.03 140.97 0)
+      (effects (font (size 1.27 1.27)) (justify bottom) hide)
+    )
+    (property "MAXIMUM_PACKAGE_HEIGHT" "2.66 mm" (at 240.03 140.97 0)
+      (effects (font (size 1.27 1.27)) (justify bottom) hide)
+    )
+    (property "MANUFACTURER" "Amphenol ICC" (at 240.03 140.97 0)
+      (effects (font (size 1.27 1.27)) (justify bottom) hide)
+    )
+    (pin "1")
+    (pin "2")
+    (pin "3")
+    (pin "4")
+    (pin "5")
+    (pin "S1")
+    (pin "S2")
+    (pin "S3")
+    (pin "S4")
+    (pin "S5")
+    (pin "S6")
+    (instances
+      (project "ESP-ExtBoard"
+        (path "/1974cf77-3075-4097-b9ae-5746e4e11ede"
+          (reference "J6") (unit 1)
+        )
+      )
+    )
   )
   (symbol (lib_id "New_Library:PIN_HEADER_1x4") (at 124.46 52.07 90) (unit 1)
@@
         (path "/1974cf77-3075-4097-b9ae-5746e4e11ede"
           (reference "U2") (unit 1)
+        )
+      )
+    )
+  )
+  (symbol (lib_id "Regulator_Linear:AMS1117-3.3") (at 215.9 128.27 0) (unit 1)
+    (in_bom yes) (on_board yes) (dnp no) (fields_autoplaced)
+    (property "Reference" "U7" (at 215.9 121.92 0)
+      (effects (font (size 1.27 1.27)))
+    )
+    (property "Value" "AMS1117-3.3" (at 215.9 124.46 0)
+      (effects (font (size 1.27 1.27)))
+    )
+    (property "Footprint" "Package_TO_SOT_SMD:SOT-223-3_TabPin2" (at 215.9 123.19 0)
+      (effects (font (size 1.27 1.27)) hide)
+    )
+    (property "Datasheet" "http://www.advanced-monolithic.com/pdf/ds1117.pdf" (at 218.44 134.62 0)
+      (effects (font (size 1.27 1.27)) hide)
+    )
+    (pin "1")
+    (pin "2")
+    (pin "3")
+    (instances
+      (project "ESP-ExtBoard"
+        (path "/1974cf77-3075-4097-b9ae-5746e4e11ede"
+          (reference "U7") (unit 1)
         )
       )
@@
     )
   )
+  (symbol (lib_id "New_Library:CH340C") (at 187.96 88.9 0) (unit 1)
+    (in_bom yes) (on_board yes) (dnp no) (fields_autoplaced)
+    (property "Reference" "U6" (at 187.96 63.5 0)
+      (effects (font (size 1.27 1.27)))
+    )
+    (property "Value" "CH340C" (at 187.96 66.04 0)
+      (effects (font (size 1.27 1.27)))
+    )
+    (property "Footprint" "New_lib:SOIC127P600X180-16N" (at 187.96 88.9 0)
+      (effects (font (size 1.27 1.27)) (justify bottom) hide)
+    )
+    (property "Datasheet" "" (at 187.96 88.9 0)
+      (effects (font (size 1.27 1.27)) hide)
+    )
+    (property "PARTREV" "2G" (at 187.96 88.9 0)
+      (effects (font (size 1.27 1.27)) (justify bottom) hide)
+    )
+    (property "STANDARD" "IPC 7351B" (at 187.96 88.9 0)
+      (effects (font (size 1.27 1.27)) (justify bottom) hide)
+    )
+    (property "MAXIMUM_PACKAGE_HEIGHT" "1.8 mm" (at 187.96 88.9 0)
+      (effects (font (size 1.27 1.27)) (justify bottom) hide)
+    )
+    (property "MANUFACTURER" "WCH" (at 187.96 88.9 0)
+      (effects (font (size 1.27 1.27)) (justify bottom) hide)
+    )
+    (pin "1")
+    (pin "10")
+    (pin "11")
+    (pin "12")
+    (pin "13")
+    (pin "14")
+    (pin "15")
+    (pin "16")
+    (pin "2")
+    (pin "3")
+    (pin "4")
+    (pin "5")
+    (pin "6")
+    (pin "7")
+    (pin "8")
+    (pin "9")
+    (instances
+      (project "ESP-ExtBoard"
+        (path "/1974cf77-3075-4097-b9ae-5746e4e11ede"
+          (reference "U6") (unit 1)
+        )
+      )
+    )
+  )
   (symbol (lib_id "power:Earth") (at 115.57 133.35 270) (unit 1)
     (in_bom yes) (on_board yes) (dnp no) (fields_autoplaced)
@@
     )
   )
+  (symbol (lib_id "New_Library:502570-0893") (at 187.96 130.81 0) (unit 1)
+    (in_bom yes) (on_board yes) (dnp no) (fields_autoplaced)
+    (property "Reference" "J5" (at 187.96 113.03 0)
+      (effects (font (size 1.27 1.27)))
+    )
+    (property "Value" "502570-0893" (at 187.96 115.57 0)
+      (effects (font (size 1.27 1.27)))
+    )
+    (property "Footprint" "New_lib:MOLEX_502570-0893" (at 187.96 130.81 0)
+      (effects (font (size 1.27 1.27)) (justify bottom) hide)
+    )
+    (property "Datasheet" "" (at 187.96 130.81 0)
+      (effects (font (size 1.27 1.27)) hide)
+    )
+    (pin "1")
+    (pin "2")
+    (pin "3")
+    (pin "4")
+    (pin "5")
+    (pin "6")
+    (pin "7")
+    (pin "8")
+    (pin "DL")
+    (pin "DS")
+    (instances
+      (project "ESP-ExtBoard"
+        (path "/1974cf77-3075-4097-b9ae-5746e4e11ede"
+          (reference "J5") (unit 1)
+        )
+      )
+    )
+  )
   (symbol (lib_id "power:Earth") (at 114.3 149.86 270) (unit 1)
     (in_bom yes) (on_board yes) (dnp no) (fields_autoplaced)
@@
         )
       )
+    )
+  )
+  (symbol (lib_id "RF_Module:ESP32-WROOM-32") (at 71.12 156.21 0) (unit 1)
+    (in_bom yes) (on_board yes) (dnp no) (fields_autoplaced)
+    (property "Reference" "U5" (at 73.0759 118.11 0)
+      (effects (font (size 1.27 1.27)) (justify left))
+    )
+    (property "Value" "ESP32-WROOM-32" (at 73.0759 120.65 0)
+      (effects (font (size 1.27 1.27)) (justify left))
+    )
+    (property "Footprint" "RF_Module:ESP32-WROOM-32" (at 71.12 194.31 0)
+      (effects (font (size 1.27 1.27)) hide)
+    )
+    (property "Datasheet" "https://www.espressif.com/sites/default/files/documentation/esp32-wroom-32_datasheet_en.pdf" (at 63.5 154.94 0)
+      (effects (font (size 1.27 1.27)) hide)
+    )
+    (pin "1")
+    (pin "10")
+    (pin "11")
+    (pin "12")
+    (pin "13")
+    (pin "14")
+    (pin "15")
+    (pin "16")
+    (pin "17")
+    (pin "18")
+    (pin "19")
+    (pin "2")
+    (pin "20")
+    (pin "21")
+    (pin "22")
+    (pin "23")
+    (pin "24")
+    (pin "25")
+    (pin "26")
+    (pin "27")
+    (pin "28")
+    (pin "29")
+    (pin "3")
+    (pin "30")
+    (pin "31")
+    (pin "32")
+    (pin "33")
+    (pin "34")
+    (pin "35")
+    (pin "36")
+    (pin "37")
+    (pin "38")
+    (pin "39")
+    (pin "4")
+    (pin "5")
+    (pin "6")
+    (pin "7")
+    (pin "8")
+    (pin "9")
+    (instances
+      (project "ESP-ExtBoard"
+        (path "/1974cf77-3075-4097-b9ae-5746e4e11ede"
+          (reference "U5") (unit 1)
+        )
+      )

Commit message: Added GPS Module
Parts:
- removed J1: PIN_HEADER, New_lib:PinHeader_1x06_P2.54mm_Vertical_1, symbol New_Library:SD_Module
- removed J2: PIN_HEADER_1x4, New_lib:PinHeader_1x04_P2.54mm_Vertical_1, symbol New_Library:PIN_HEADER_1x4
- removed U1: ESP32-DEVKIT-V1, New_lib:MODULE_ESP32_DEVKIT_V1, symbol New_Library:ESP32-DEVKIT-V1
- added J1: NEO-GPS, New_lib:NEO-GPS, symbol New_Library:NEO-GPS
Connections:
- net +3.3V: now also U5.2 (VDD), U6.16 (VCC), U7.2 (VO), J1.1 (VCC)
- net Earth: now also U5.1 (GND), U5.15 (GND), U5.38 (GND), U5.39 (GND), U7.1 (GND), J1.4 (GND)
- net GPIO14: now also U5.13 (IO14)
- net GPIO25: now also U5.10 (IO25)
- net GPIO26: now also U5.11 (IO26)
- net GPIO27: now also U5.12 (IO27)
- net GPIO32: now also U5.8 (IO32)
- net GPIO33: now also U5.9 (IO33)
- net GPIO34: now also U5.6 (IO34)
- net GPIO35: now also U5.7 (IO35)
- net I2C0_SCL: now also U5.36 (IO22)
- net I2C0_SDA: now also U5.33 (IO21)
- net UART2_RX: now also U5.27 (IO16), J1.3 (TX)
- net UART2_TX: now also U5.28 (IO17), J1.2 (RX)
- net VSPI_CLK: now also U5.30 (IO18)
- net VSPI_CS: now also U5.29 (IO5)
- net VSPI_MISO: now also U5.31 (IO19)
- net VSPI_MOSI: now also U5.37 (IO23)
- net UART0_TX: now reaches U6.2 (TXD)
- net UART0_TX: now also U5.35 (TXD0/IO1)
- net UART0_RX: now reaches U6.3 (RXD)
- net UART0_RX: now also U5.34 (RXD0/IO3)
Other:
- moved on the sheet: J3, J4, U5, U7
